File: case/PCB_Front/front.kicad_pcb (KiCad board)
At the start: 2 copper layers, 164 x 142 mm, 2 parts

Commit message: kicad stuff v1
Parts:
- removed the G*** at (0.00, 0.00) (x2)
- added G*** (x2): LOGO, LOGO, F.Cu at (0.00, 0.00)
Changed lines of the file:
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@@
     (visible_elements 7FFFFFFF)
     (pcbplotparams
-      (layerselection 0x010f0_80000001)
+      (layerselection 0x010f0_ffffffff)
       (usegerberextensions false)
       (usegerberattributes false)
@@
       (outputformat 1)
       (mirror false)
-      (drillshape 1)
+      (drillshape 0)
       (scaleselection 1)
       (outputdirectory "gerbers/"))

Commit message: v2 backboard
Parts:
- removed the G*** at (0.00, 0.00) (x2)
- added G*** (x2): LOGO, LOGO, F.Cu at (0.00, 0.00)
Other:
- outline, holes or cut-outs redrawn
